Commit message: change Moveit config to DexWrist gripper

File: stretch_moveit2/stretch_moveit_config/config/stretch_arm.ros2_control.xacro (robot description, xacro)
@@ -42,4 +42,16 @@
                 <state_interface name="velocity"/>
             </joint>
+            <joint name="joint_wrist_roll">
+                <param name="initial_position">0.0</param>
+                <command_interface name="position" />
+                <state_interface name="position"/>
+                <state_interface name="velocity"/>
+            </joint>
+            <joint name="joint_wrist_pitch">
+                <param name="initial_position">0.0</param>
+                <command_interface name="position" />
+                <state_interface name="position"/>
+                <state_interface name="velocity"/>
+            </joint>
         </ros2_control>
     </xacro:macro>
